File: PCB/blanking/blanking.sch (KiCad schematic (older format))
At the start: 25 parts, among them J1 Conn_01x03_Male, J10 Conn_01x03_Male, J11 Conn_01x03_Male, J12 Conn_01x03_Male, J13 PWM_controls_driver, J2 Conn_01x03_Male, J3 Conn_01x03_Male, J4 Conn_01x07, J5 Conn_02x07_Odd_Even, J6 Conn_01x03_Male, J7 Conn_01x03_Male, J8 Conn_01x03_Male, J9 blanking, Q1 Q_PNP_EBC, Q2 Q_PNP_EBC, Q3 Q_PNP_EBC, Q4 Q_PNP_EBC, Q5 Q_PNP_EBC, Q6 Q_PNP_EBC, U1 4069

Commit message: update pcbs for production
Parts:
- removed J4: Conn_01x07, Connectors_Molex:Molex_KK-6410-07_07x2.54mm_Straight, symbol Conn_01x07
- removed U1: 4069, symbol 4069
- added J14: vcc_inverters, Connectors:PINHEAD1-2, symbol conn:Conn_01x02
- added R5, R6: R, Resistors_THT:R_Axial_DIN0204_L3.6mm_D1.6mm_P2.54mm_Vertical, symbol Device:R
- added U1, U3: 74AHC1G14, Housings_SSOP:TSOP-5_1.65x3.05mm_Pitch0.95mm, symbol blanking-rescue:74AHC1G14
- J1: value Conn_01x03_Male -> inverter/non_inverter3; symbol Conn_01x03_Male -> conn:Conn_01x03_Male
- J10: value Conn_01x03_Male -> blank/nonblank2; symbol Conn_01x03_Male -> conn:Conn_01x03_Male; Field4 (none) -> blanking_select
- J11: value Conn_01x03_Male -> blank/nonblank3; symbol Conn_01x03_Male -> conn:Conn_01x03_Male
- J12: value Conn_01x03_Male -> blank/non_blank1; symbol Conn_01x03_Male -> conn:Conn_01x03_Male
- J13: symbol Screw_Terminal_01x04 -> conn:Screw_Terminal_01x04
- J2: value Conn_01x03_Male -> inverter/non_inverter1; symbol Conn_01x03_Male -> conn:Conn_01x03_Male
- J3: value Conn_01x03_Male -> inverter/non_inverter2; symbol Conn_01x03_Male -> conn:Conn_01x03_Male
- J5: value Conn_02x07_Odd_Even -> to_LCr_J29; symbol Conn_02x07_Odd_Even -> conn:Conn_02x07_Odd_Even
- J6: value Conn_01x03_Male -> enab/non_enab3; symbol Conn_01x03_Male -> conn:Conn_01x03_Male
- J7: value Conn_01x03_Male -> enab/no_enab2; symbol Conn_01x03_Male -> conn:Conn_01x03_Male
- J8: value Conn_01x03_Male -> enable/non_enbale1; symbol Conn_01x03_Male -> conn:Conn_01x03_Male
- J9: symbol Screw_Terminal_01x02 -> conn:Screw_Terminal_01x02
- Q1, Q4: symbol Q_PNP_EBC -> Device:Q_PNP_EBC
- Q2: value Q_PNP_EBC -> enab/nonenab2_PNP_EBC; symbol Q_PNP_EBC -> Device:Q_PNP_EBC
- Q3: symbol Q_PNP_EBC -> Device:Q_PNP_EBC; Field4 (none) -> enable_pwm
- Q5: symbol Q_PNP_EBC -> Device:Q_PNP_EBC; Field4 (none) -> pwm_blank
- Q6: value Q_PNP_EBC -> blank_trans3_PNP_EBC; symbol Q_PNP_EBC -> Device:Q_PNP_EBC
- R1, R2, R3, R4: symbol R -> Device:R
- U2: renamed from U?; footprint (none) -> Housings_SSOP:TSOP-5_1.65x3.05mm_Pitch0.95mm; symbol 74AHC1G14 -> blanking-rescue:74AHC1G14
Connections:
- wire segments 146 -> 181
Other:
- moved on the sheet: J1, J10, J11, J12, J13, J2, J3, J5, J6, J7, J8, J9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
