File: PCB/blanking/blanking.kicad_pcb (KiCad board)
At the start: 2 copper layers, 95.5 x 42.5 mm, 32 parts, among them J10_red_blank non_blank/blank 2, J11_blue_blank non_blank/blank3, J12_green_blank non_blank/blank 1, J13 PWM_controls_driver, J14_inv_vcc inv_vcc, J1_Blue_enab non_inv/inv 3, J2_Green_PWM non_inv/inv 1, J3_Red_PWM non_inv/inv 2, J5 to_LCr_J29, J6_Blue_Enab Conn_01x03_Male blue, J7_Red_enab Conn_01x03_Male, J8_Green_Enab Conn_01x03_Male, J9 blanking, Q1 Q_PNP_EBC, Q2 Q_PNP_EBC, Q3 Q_PNP_EBC, Q4 Q_PNP_EBC, Q5 Q_PNP_EBC, Q6 Q_PNP_EBC, U1 Inverter 3, U2 inverter2, U3 inverter1

Commit message: update to PCBs
Routing:
- net Net-(J14-Pad1): track 94.2 -> 80.1 mm
Changed lines of the file:
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@@
       (effects (font (size 1 1) (thickness 0.15)))
     )
-    (fp_text value MountingHole_3.2mm_M3 (at 0 4.2) (layer F.Fab)
+    (fp_text value MountingHole_3.2mm_M3 (at 0 4) (layer F.Fab)
       (effects (font (size 1 1) (thickness 0.15)))
     )
@@
     (pad 1 np_thru_hole circle (at 0 0) (size 3.2 3.2) (drill 3.2) (layers *.Cu *.Mask))
   )
-  (target plus (at 173.45 83.275) (size 5) (width 0.15) (layer Edge.Cuts))
+  (target plus (at 184.35879 78.906288) (size 5) (width 0.15) (layer Edge.Cuts))
   (gr_text BRG- (at 183.7 64.025 90) (layer F.SilkS)
     (effects (font (size 1.5 1.5) (thickness 0.3)))
@@
   (segment (start 255.45 79.525) (end 247.1 79.525) (width 0.25) (layer F.Cu) (net 29))
   (segment (start 247.1 79.525) (end 243.75 82.875) (width 0.25) (layer F.Cu) (net 29))
-  (segment (start 215.95 82.875) (end 215.35 82.275) (width 0.25) (layer F.Cu) (net 29))
-  (segment (start 243.75 82.875) (end 215.95 82.875) (width 0.25) (layer F.Cu) (net 29))
+  (segment (start 230.075002 82.875) (end 229.475002 82.275) (width 0.25) (layer F.Cu) (net 29))
+  (segment (start 243.75 82.875) (end 230.075002 82.875) (width 0.25) (layer F.Cu) (net 29))
   (segment (start 233.790001 68.575001) (end 233.790001 68.315001) (width 0.25) (layer F.Cu) (net 30))
   (segment (start 230.7 65.315) (end 232.95 63.065) (width 0.25) (layer F.Cu) (net 30))
