File: PCB/uvled/uv_led.kicad_pcb (KiCad board)
At the start: 2 copper layers, 2 parts, among them J1 Conn_01x02_Female

Commit message: update uv board
Other:
- board outline added: 25 x 25 mm
Changed lines of the file:
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@@
-(kicad_pcb (version 4) (host pcbnew 4.0.7)
+(kicad_pcb (version 20171130) (host pcbnew "(5.0.0)")
   (general
-    (links 4)
-    (no_connects 0)
-    (area 135.899999 81.399999 161.100001 106.600001)
     (thickness 1.6)
     (drawings 6)
@@
     (trace_min 0.2)
     (segment_width 0.2)
-    (edge_width 0.15)
+    (edge_width 0.2)
     (via_size 0.6)
     (via_drill 0.4)
@@
     (pad_drill 0.762)
     (pad_to_mask_clearance 0.2)
-    (aux_axis_origin 142 101)
-    (visible_elements FFFFFF7F)
+    (aux_axis_origin 142.05 100.975)
+    (visible_elements 7FFFFFFF)
     (pcbplotparams
-      (layerselection 0x03830_80000001)
+      (layerselection 0x03830_ffffffff)
       (usegerberextensions false)
+      (usegerberattributes false)
+      (usegerberadvancedattributes false)
+      (creategerberjobfile false)
       (excludeedgelayer true)
       (linewidth 0.100000)
@@
       (hpglpennumber 1)
       (hpglpenspeed 20)
-      (hpglpendiameter 15)
-      (hpglpenoverlay 2)
+      (hpglpendiameter 15.000000)
       (psnegative false)
       (psa4output false)
@@
       (drillshape 0)
       (scaleselection 1)
-      (outputdirectory ""))
+      (outputdirectory "gerber/"))
   )
   (net 0 "")
@@
       (net 2 +3V3))
     (model ${KISYS3DMOD}/Socket_Strips.3dshapes/Socket_Strip_Straight_1x02_Pitch2.54mm.wrl
-      (at (xyz 0 -0.05 0))
+      (offset (xyz 0 -1.269999980926514 0))
       (scale (xyz 1 1 1))
       (rotate (xyz 0 0 270))
     )
   )
-  (target plus (at 142 101) (size 5) (width 0.15) (layer Edge.Cuts))
+  (target plus (at 142.025 101) (size 5) (width 0.2) (layer Edge.Cuts))
   (gr_text - (at 147 84) (layer B.SilkS)
     (effects (font (size 1.5 1.5) (thickness 0.3)))
@@
     (effects (font (size 1.5 1.5) (thickness 0.3)))
   )
-  (gr_circle (center 148.5 94) (end 148.5 106.5) (layer Eco2.User) (width 0.2))
+  (gr_circle (center 148.5 94) (end 161 94) (layer Edge.Cuts) (width 0.2))
   (segment (start 153.59126 93.98) (end 151.003 93.98) (width 0.75) (layer F.Cu) (net 2))
   (segment (start 151.003 93.98) (end 151.003 91.003) (width 0.75) (layer F.Cu) (net 2))
